Commit message: add config for multirobot (in progress)

File: src/jackal_description/urdf/accessories/OS1-32.urdf.xacro (robot description, xacro)
@@ -2,18 +2,25 @@
 <robot xmlns:xacro="http://www.ros.org/wiki/xacro">
   <xacro:property name="M_PI" value="3.1415926535897931" />
-  <xacro:macro name="OS1-32" params="*origin parent:=base_link name:=os_sensor topic_points:=/ouster/points topic_imu:=/ouster/imu hz:=10 lasers:=32 samples:=1024 min_range:=0.3 max_range:=75.0 noise:=0.008 min_angle:=-${M_PI} max_angle:=${M_PI} lidar_link:=os_lidar imu_link:=os_imu vfov_min:=-.393 vfov_max:=.393">
-  <!-- <xacro:macro name="OS1-32" params="*origin parent:=base_link name:=os_sensor"> -->
+  <xacro:macro name="OS1-32" params="*origin parent:=base_link name:=os_sensor topic_points:=/ouster/points topic_imu:=/ouster/imu hz:=10 lasers:=32 samples:=1024 min_range:=0.3 max_range:=75.0 noise:=0.008 min_angle:=-${M_PI} max_angle:=${M_PI} lidar_link:=os_lidar imu_link:=os_imu vfov_min:=-.393 vfov_max:=.393 namespace:=''">
+    <xacro:property name="ns_value" value="$(arg namespace)" />
+    <xacro:property name="lidar_link_ns" value="${lidar_link}" />
+    <!-- <xacro:unless value="$(arg namespace)">
+      <xacro:property name="lidar_link_ns" value="${lidar_link_ns}" />
+    </xacro:unless> -->
+    <xacro:if value="${ns_value != ''}">
+      <xacro:property name="lidar_link_ns" value="$(arg namespace)/${lidar_link}" />
+    </xacro:if>
     <joint name="${name}_mount_joint" type="fixed">
       <xacro:insert_block name="origin" />
-      <parent link="${parent}"/>
-      <child link="${name}_base_link"/>
+      <parent link="$(arg namespace)/${parent}"/>
+      <child link="$(arg namespace)/${name}_base_link"/>
     </joint>
-    <link name="${name}_base_link" />
+    <link name="$(arg namespace)/${name}_base_link" />
     <joint name="${name}_base_to_baseplate" type="fixed">
-      <parent link="${name}_base_link"/>
-      <child link="${name}_baseplate" />
+      <parent link="$(arg namespace)/${name}_base_link"/>
+      <child link="$(arg namespace)/${name}_baseplate" />
       <origin xyz="0 0 0.008"/>
     </joint>
-    <link name="${name}_baseplate">
+    <link name="$(arg namespace)/${name}_baseplate">
       <visual>
         <geometry>
@@ -31,9 +38,9 @@
     </link>
     <joint name="${name}_baseplate_to_body" type="fixed">
-      <parent link="${name}_baseplate"/>
-      <child link="${name}"/>
+      <parent link="$(arg namespace)/${name}_baseplate"/>
+      <child link="$(arg namespace)/${name}"/>
       <origin xyz="0 0 0.042" rpy="0 0 0" />
     </joint>
-    <link name="${name}">
+    <link name="$(arg namespace)/${name}">
       <inertial>
          <mass value="0.33"/>
@@ -56,28 +63,28 @@
       </visual>
     </link>
-    <link name="${imu_link}" />
-    <link name="${lidar_link}" />
+    <link name="$(arg namespace)/${imu_link}" />
+    <link name="${lidar_link_ns}" />
     <joint name="${name}_imu_link_joint" type="fixed">
-      <parent link="${name}" />
-      <child link="${imu_link}" />
+      <parent link="$(arg namespace)/${name}" />
+      <child link="$(arg namespace)/${imu_link}" />
       <origin xyz="0.006253 -0.011775 0.007645" rpy="0 0 0" />
     </joint>
-    <gazebo reference="${imu_link}">
+    <gazebo reference="$(arg namespace)/${imu_link}">
     </gazebo>
     <joint name="${name}_lidar_link_joint" type="fixed">
-      <parent link="${name}" />
-      <child link="${lidar_link}" />
+      <parent link="$(arg namespace)/${name}" />
+      <child link="${lidar_link_ns}" />
       <origin xyz="0.0 0.0 0.03618" rpy="0 0 0" />
     </joint>
     <!-- Gazebo requires the ouster_gazebo_plugins package -->
-    <gazebo reference="${name}">
+    <gazebo reference="$(arg namespace)/${name}">
         <selfCollide>false</selfCollide>
-        <sensor name="${name}-OS1-32" type="gpu_lidar">
+        <sensor name="$(arg namespace)/${name}-OS1-32" type="gpu_lidar">
             <pose> 0 0 0 0 0 0 </pose>
             <always_on>true</always_on>
             <update_rate>${hz}</update_rate>
             <visualize>false</visualize>
-            <gz_frame_id>${lidar_link}</gz_frame_id>
-            <topic>${topic_points}</topic>
+            <gz_frame_id>${lidar_link_ns}</gz_frame_id>
+            <topic>$(arg namespace)${topic_points}</topic>
             <lidar>
                 <scan>

File: src/jackal_description/urdf/accessories/_d435.urdf.xacro (robot description, xacro)
@@ -51,14 +51,14 @@
     <joint name="${name}_joint" type="fixed">
       <xacro:insert_block name="origin" />
-      <parent link="${parent}"/>
-      <child link="${name}_bottom_screw_frame" />
+      <parent link="$(arg namespace)/${parent}"/>
+      <child link="$(arg namespace)/${name}_bottom_screw_frame" />
     </joint>
-    <link name="${name}_bottom_screw_frame"/>
+    <link name="$(arg namespace)/${name}_bottom_screw_frame"/>
     <joint name="${name}_link_joint" type="fixed">
       <origin xyz="${d435_mesh_x_offset} ${d435_cam_depth_py} ${d435_cam_depth_pz}" rpy="0 0 0"/>
-      <parent link="${name}_bottom_screw_frame"/>
-      <child link="${name}_link" />
+      <parent link="$(arg namespace)/${name}_bottom_screw_frame"/>
+      <child link="$(arg namespace)/${name}_link" />
     </joint>
-    <link name="${name}_link">
+    <link name="$(arg namespace)/${name}_link">
       <visual>
         <xacro:if value="${use_mesh}">
@@ -96,53 +96,53 @@
       <joint name="${name}_depth_joint" type="fixed">
         <origin xyz="0 0 0" rpy="0 0 0"/>
-        <parent link="${name}_link"/>
-        <child link="${name}_depth_frame" />
+        <parent link="$(arg namespace)/${name}_link"/>
+        <child link="$(arg namespace)/${name}_depth_frame" />
       </joint>
-      <link name="${name}_depth_frame"/>
+      <link name="$(arg namespace)/${name}_depth_frame"/>
       <joint name="${name}_depth_optical_joint" type="fixed">
         <origin xyz="0 0 0" rpy="${-M_PI/2} 0 ${-M_PI/2}" />
-        <parent link="${name}_depth_frame" />
-        <child link="${name}_depth_optical_frame" />
+        <parent link="$(arg namespace)/${name}_depth_frame" />
+        <child link="$(arg namespace)/${name}_depth_optical_frame" />
       </joint>
-      <link name="${name}_depth_optical_frame"/>
+      <link name="$(arg namespace)/${name}_depth_optical_frame"/>
       <!-- camera left IR joints and links -->
       <joint name="${name}_infra1_joint" type="fixed">
         <origin xyz="0 ${d435_cam_depth_to_infra1_offset} 0" rpy="0 0 0" />
-        <parent link="${name}_link" />
-        <child link="${name}_infra1_frame" />
+        <parent link="$(arg namespace)/${name}_link" />
+        <child link="$(arg namespace)/${name}_infra1_frame" />
       </joint>
-      <link name="${name}_infra1_frame"/>
+      <link name="$(arg namespace)/${name}_infra1_frame"/>
       <joint name="${name}_infra1_optical_joint" type="fixed">
         <origin xyz="0 0 0" rpy="${-M_PI/2} 0 ${-M_PI/2}" />
-        <parent link="${name}_infra1_frame" />
-        <child link="${name}_infra1_optical_frame" />
+        <parent link="$(arg namespace)/${name}_infra1_frame" />
+        <child link="$(arg namespace)/${name}_infra1_optical_frame" />
       </joint>
-      <link name="${name}_infra1_optical_frame"/>
+      <link name="$(arg namespace)/${name}_infra1_optical_frame"/>
       <!-- camera right IR joints and links -->
       <joint name="${name}_infra2_joint" type="fixed">
         <origin xyz="0 ${d435_cam_depth_to_infra2_offset} 0" rpy="0 0 0" />
-        <parent link="${name}_link" />
-        <child link="${name}_infra2_frame" />
+        <parent link="$(arg namespace)/${name}_link" />
+        <child link="$(arg namespace)/${name}_infra2_frame" />
       </joint>
-      <link name="${name}_infra2_frame"/>
+      <link name="$(arg namespace)/${name}_infra2_frame"/>
       <joint name="${name}_infra2_optical_joint" type="fixed">
         <origin xyz="0 0 0" rpy="${-M_PI/2} 0 ${-M_PI/2}" />
-        <parent link="${name}_infra2_frame" />
-        <child link="${name}_infra2_optical_frame" />
+        <parent link="$(arg namespace)/${name}_infra2_frame" />
+        <child link="$(arg namespace)/${name}_infra2_optical_frame" />
       </joint>
-      <link name="${name}_infra2_optical_frame"/>
+      <link name="$(arg namespace)/${name}_infra2_optical_frame"/>
       <!-- camera color joints and links -->
       <joint name="${name}_color_joint" type="fixed">
         <origin xyz="0 ${d435_cam_depth_to_color_offset} 0" rpy="0 0 0" />
-        <parent link="${name}_link" />
-        <child link="${name}_color_frame" />
+        <parent link="$(arg namespace)/${name}_link" />
+        <child link="$(arg namespace)/${name}_color_frame" />
       </joint>
-      <link name="${name}_color_frame"/>
+      <link name="$(arg namespace)/${name}_color_frame"/>
       <joint name="${name}_color_optical_joint" type="fixed">
         <origin xyz="0 0 0" rpy="${-M_PI/2} 0 ${-M_PI/2}" />
-        <parent link="${name}_color_frame" />
-        <child link="${name}_color_optical_frame" />
+        <parent link="$(arg namespace)/${name}_color_frame" />
+        <child link="$(arg namespace)/${name}_color_optical_frame" />
       </joint>
-      <link name="${name}_color_optical_frame"/>
+      <link name="$(arg namespace)/${name}_color_optical_frame"/>
     </xacro:if>
     <xacro:if value="${add_plug}">

File: src/jackal_description/urdf/accessories/_usb_plug.urdf.xacro (robot description, xacro)
@@ -24,8 +24,8 @@
     <joint name="${name}_joint" type="fixed">
       <xacro:insert_block name="origin" />
-      <parent link="${parent}" />
-      <child link="${name}_link" />
+      <parent link="$(arg namespace)/${parent}" />
+      <child link="$(arg namespace)/${name}_link" />
     </joint>
-    <link name="${name}_link">
+    <link name="$(arg namespace)/${name}_link">
       <visual>
         <!-- 0.044850 0.008000 0.018500 -->

File: src/jackal_description/urdf/accessories/camera_mount.urdf.xacro (robot description, xacro)
@@ -1,5 +1,5 @@
 <robot xmlns:xacro="http://www.ros.org/wiki/xacro">
   <xacro:macro name="camera_mount" params="prefix tilt:=0">
-    <link name="${prefix}_camera_mount">
+    <link name="$(arg namespace)/${prefix}_camera_mount">
       <visual>
         <origin xyz="0 0 0" rpy="1.5707 0 1.5707" />
@@ -10,5 +10,5 @@
       </visual>
     </link>
-    <link name="${prefix}_camera_beam">
+    <link name="$(arg namespace)/${prefix}_camera_beam">
       <visual>
         <origin xyz="0 0 0" rpy="0 0 1.5707" />
@@ -21,11 +21,11 @@
     <joint name="${prefix}_camera_pivot_joint" type="fixed">
       <origin xyz="0.102 0 0.008" rpy="0 ${tilt} 0" />
-      <parent link="${prefix}_camera_mount" />
-      <child link="${prefix}_camera_beam" />
+      <parent link="$(arg namespace)/${prefix}_camera_mount" />
+      <child link="$(arg namespace)/${prefix}_camera_beam" />
     </joint>
-    <gazebo reference="${prefix}_camera_beam">
+    <gazebo reference="$(arg namespace)/${prefix}_camera_beam">
       <material>Gazebo/DarkGrey</material>
     </gazebo>
-    <gazebo reference="${prefix}_camera_mount">
+    <gazebo reference="$(arg namespace)/${prefix}_camera_mount">
       <material>Gazebo/DarkGrey</material>
     </gazebo>

File: src/jackal_description/urdf/jackal.urdf.xacro (robot description, xacro)
@@ -2,4 +2,5 @@
 <robot name="jackal" xmlns:xacro="http://www.ros.org/wiki/xacro">
   <xacro:property name="PI" value="3.1415926535897931" />
+  <xacro:arg name="namespace" default='' />
   <!-- Jackal properties -->
   <xacro:property name="wheelbase" value="0.262" />
@@ -20,5 +21,5 @@
   <!-- Wheels macro -->
   <xacro:macro name="wheel" params="prefix mu *joint_pose">
-    <link name="${prefix}_wheel_link">
+    <link name="$(arg namespace)/${prefix}_wheel_link">
       <visual>
         <origin xyz="0 0 0" rpy="${PI/2} 0 0"/>
@@ -44,6 +45,6 @@
     </link>
     <joint name="${prefix}_wheel" type="continuous">
-      <parent link="chassis_link"/>
-      <child link="${prefix}_wheel_link" />
+      <parent link="$(arg namespace)/chassis_link"/>
+      <child link="$(arg namespace)/${prefix}_wheel_link" />
       <xacro:insert_block name="joint_pose" />
       <axis xyz="0 1 0" />
@@ -60,11 +61,11 @@
   </xacro:macro>
   <!-- Links and joints -->
-  <link name="base_link"></link>
+  <link name="$(arg namespace)/base_link"></link>
   <joint name="base_link_joint" type="fixed">
     <origin xyz="0 0 0" rpy="0 0 0" />
-    <parent link="base_link"/>
-    <child link="chassis_link" />
-  </joint>
-  <link name="chassis_link">
+    <parent link="$(arg namespace)/base_link"/>
+    <child link="$(arg namespace)/chassis_link" />
+  </joint>
+  <link name="$(arg namespace)/chassis_link">
     <visual>
       <origin xyz="0 0 ${footprint_vertical_offset}" rpy="${PI/2} 0 ${PI/2}"/>
@@ -89,5 +90,5 @@
       </inertial>
   </link>
-  <link name="front_fender_link">
+  <link name="$(arg namespace)/front_fender_link">
     <visual>
       <geometry>
@@ -97,16 +98,16 @@
     </visual>
   </link>
-  <link name="front_fender_accessory_link"/>
+  <link name="$(arg namespace)/front_fender_accessory_link"/>
   <joint name="front_fender_accessory_joint" type="fixed">
     <origin xyz="0.25629 0 0.07455" rpy="${PI} 0 0" />
-    <parent link="front_fender_link" />
-    <child link="front_fender_accessory_link" />
+    <parent link="$(arg namespace)/front_fender_link" />
+    <child link="$(arg namespace)/front_fender_accessory_link" />
   </joint>
   <joint name="front_fender_joint" type="fixed">
     <origin xyz="0 0 0" rpy="0 0 0"/>
-    <parent link="chassis_link" />
-    <child link="front_fender_link" />
-  </joint>
-  <link name="rear_fender_link">
+    <parent link="$(arg namespace)/chassis_link" />
+    <child link="$(arg namespace)/front_fender_link" />
+  </joint>
+  <link name="$(arg namespace)/rear_fender_link">
     <visual>
       <geometry>
@@ -116,14 +117,14 @@
     </visual>
   </link>
-  <link name="rear_fender_accessory_link"/>
+  <link name="$(arg namespace)/rear_fender_accessory_link"/>
   <joint name="rear_fender_accessory_joint" type="fixed">
     <origin xyz="0.25629 0 0.07455" rpy="${PI} 0 0" />
-    <parent link="rear_fender_link" />
-    <child link="rear_fender_accessory_link" />
+    <parent link="$(arg namespace)/rear_fender_link" />
+    <child link="$(arg namespace)/rear_fender_accessory_link" />
   </joint>
   <joint name="rear_fender_joint" type="fixed">
     <origin xyz="0 0 0" rpy="0 0 ${PI}"/>
-    <parent link="chassis_link" />
-    <child link="rear_fender_link" />
+    <parent link="$(arg namespace)/chassis_link" />
+    <child link="$(arg namespace)/rear_fender_link" />
   </joint>
   <!-- Wheels links and joints -->
@@ -141,5 +142,5 @@
   </xacro:wheel>
   <!-- Default Internal IMU Link -->
-  <link name="imu_link">
+  <link name="$(arg namespace)/imu_link">
     <inertial>
       <mass value="0.001"/>
@@ -149,9 +150,9 @@
   </link>
   <joint name="imu_joint" type="fixed">
-    <parent link="chassis_link" />
-    <child link="imu_link" />
+    <parent link="$(arg namespace)/chassis_link" />
+    <child link="$(arg namespace)/imu_link" />
   </joint>
   <!-- Default NAVSAT Link -->
-  <link name="navsat_link">
+  <link name="$(arg namespace)/navsat_link">
     <visual>
       <geometry>
@@ -163,24 +164,24 @@
   </link>
   <joint name="navsat_joint" type="fixed">
-    <parent link="chassis_link" />
-    <child link="navsat_link" />
+    <parent link="$(arg namespace)/chassis_link" />
+    <child link="$(arg namespace)/navsat_link" />
     <origin xyz="-0.180 0.126 0.1815" />
   </joint>
-  <link name="mid_mount"></link>
+  <link name="$(arg namespace)/mid_mount"></link>
   <joint name="mid_mount_joint" type="fixed">
-    <parent link="chassis_link" />
-    <child link="mid_mount" />
+    <parent link="$(arg namespace)/chassis_link" />
+    <child link="$(arg namespace)/mid_mount" />
     <origin xyz="0 0 ${chassis_height}" />
   </joint>
-  <link name="rear_mount"></link>
+  <link name="$(arg namespace)/rear_mount"></link>
   <joint name="rear_mount_joint" type="fixed">
-    <parent link="mid_mount" />
-    <child link="rear_mount" />
+    <parent link="$(arg namespace)/mid_mount" />
+    <child link="$(arg namespace)/rear_mount" />
     <origin xyz="${-mount_spacing} 0 0" />
   </joint>
-  <link name="front_mount"></link>
+  <link name="$(arg namespace)/front_mount"></link>
   <joint name="front_mount_joint" type="fixed">
-    <parent link="mid_mount" />
-    <child link="front_mount" />
+    <parent link="$(arg namespace)/mid_mount" />
+    <child link="$(arg namespace)/front_mount" />
     <origin xyz="${mount_spacing} 0 0" />
   </joint>
@@ -190,20 +191,21 @@
     <origin xyz="0 0 0"
             rpy="0 0 0" />
-    <parent link="front_mount" />
-    <child link="front_camera_mount" />
+    <parent link="$(arg namespace)/front_mount" />
+    <child link="$(arg namespace)/front_camera_mount" />
   </joint>
   <!-- Realsense D435 -->
-  <!-- <xacro:arg name="use_nominal_extrinsics" default="true"/>
+  <xacro:arg name="use_nominal_extrinsics" default="true"/>
   <xacro:arg name="add_plug" default="true" />
   <xacro:arg name="use_mesh" default="true" />
   <xacro:include filename="$(find jackal_description)/urdf/accessories/_d435.urdf.xacro" />
-  <xacro:sensor_d435 parent="front_camera_beam" use_nominal_extrinsics="$(arg use_nominal_extrinsics)" add_plug="$(arg add_plug)" use_mesh="$(arg use_mesh)">
+  <xacro:sensor_d435 parent="front_camera_beam" use_nominal_extrinsics="$(arg use_nominal_extrinsics)"
+                             name="camera" add_plug="$(arg add_plug)" use_mesh="$(arg use_mesh)">
     <origin xyz="0 0 0.04" rpy="0 0 0"/>
-  </xacro:sensor_d435> -->
+  </xacro:sensor_d435>
   <!-- Ouster OS1 32SR -->
-  <!-- <xacro:include filename="$(find jackal_description)/urdf/accessories/OS1-32.urdf.xacro" />
-  <xacro:OS1-32 parent="front_camera_mount">
+  <xacro:include filename="$(find jackal_description)/urdf/accessories/OS1-32.urdf.xacro" />
+  <xacro:OS1-32 parent="front_camera_mount" name="os_sensor">
     <origin xyz="0.0 0.0 0.10201" rpy="0 0 0"/>
-  </xacro:OS1-32> -->
+  </xacro:OS1-32>
   <!-- Gazebo plugins -->
   <xacro:include filename="$(find jackal_description)/urdf/jackal.gazebo" />
