Commit message: Refined URDF links to handle optional namespaces, avoiding leading / when unused

File: src/jackal_description/urdf/accessories/OS1-32.urdf.xacro (robot description, xacro)
@@ -2,25 +2,17 @@
 <robot xmlns:xacro="http://www.ros.org/wiki/xacro">
   <xacro:property name="M_PI" value="3.1415926535897931" />
-  <xacro:macro name="OS1-32" params="*origin parent:=base_link name:=os_sensor topic_points:=/ouster/points topic_imu:=/ouster/imu hz:=10 lasers:=32 samples:=1024 min_range:=0.3 max_range:=75.0 noise:=0.008 min_angle:=-${M_PI} max_angle:=${M_PI} lidar_link:=os_lidar imu_link:=os_imu vfov_min:=-.393 vfov_max:=.393 namespace:=''">
-    <xacro:property name="ns_value" value="$(arg namespace)" />
-    <xacro:property name="lidar_link_ns" value="${lidar_link}" />
-    <!-- <xacro:unless value="$(arg namespace)">
-      <xacro:property name="lidar_link_ns" value="${lidar_link_ns}" />
-    </xacro:unless> -->
-    <xacro:if value="${ns_value != ''}">
-      <xacro:property name="lidar_link_ns" value="$(arg namespace)/${lidar_link}" />
-    </xacro:if>
+  <xacro:macro name="OS1-32" params="*origin parent:=base_link name:=os_sensor topic_points:=ouster/points topic_imu:=ouster/imu hz:=10 lasers:=32 samples:=1024 min_range:=0.3 max_range:=75.0 noise:=0.008 min_angle:=-${M_PI} max_angle:=${M_PI} lidar_link:=os_lidar imu_link:=os_imu vfov_min:=-.393 vfov_max:=.393 namespace:=''">
     <joint name="${name}_mount_joint" type="fixed">
       <xacro:insert_block name="origin" />
-      <parent link="$(arg namespace)/${parent}"/>
-      <child link="$(arg namespace)/${name}_base_link"/>
+      <parent link="${ns}${parent}"/>
+      <child link="${ns}${name}_base_link"/>
     </joint>
-    <link name="$(arg namespace)/${name}_base_link" />
+    <link name="${ns}${name}_base_link" />
     <joint name="${name}_base_to_baseplate" type="fixed">
-      <parent link="$(arg namespace)/${name}_base_link"/>
-      <child link="$(arg namespace)/${name}_baseplate" />
+      <parent link="${ns}${name}_base_link"/>
+      <child link="${ns}${name}_baseplate" />
       <origin xyz="0 0 0.008"/>
     </joint>
-    <link name="$(arg namespace)/${name}_baseplate">
+    <link name="${ns}${name}_baseplate">
       <visual>
         <geometry>
@@ -38,9 +30,9 @@
     </link>
     <joint name="${name}_baseplate_to_body" type="fixed">
-      <parent link="$(arg namespace)/${name}_baseplate"/>
-      <child link="$(arg namespace)/${name}"/>
+      <parent link="${ns}${name}_baseplate"/>
+      <child link="${ns}${name}"/>
       <origin xyz="0 0 0.042" rpy="0 0 0" />
     </joint>
-    <link name="$(arg namespace)/${name}">
+    <link name="${ns}${name}">
       <inertial>
          <mass value="0.33"/>
@@ -63,28 +55,28 @@
       </visual>
     </link>
-    <link name="$(arg namespace)/${imu_link}" />
-    <link name="${lidar_link_ns}" />
+    <link name="${ns}${imu_link}" />
+    <link name="${ns}${lidar_link}" />
     <joint name="${name}_imu_link_joint" type="fixed">
-      <parent link="$(arg namespace)/${name}" />
-      <child link="$(arg namespace)/${imu_link}" />
+      <parent link="${ns}${name}" />
+      <child link="${ns}${imu_link}" />
       <origin xyz="0.006253 -0.011775 0.007645" rpy="0 0 0" />
     </joint>
-    <gazebo reference="$(arg namespace)/${imu_link}">
+    <gazebo reference="${ns}${imu_link}">
     </gazebo>
     <joint name="${name}_lidar_link_joint" type="fixed">
-      <parent link="$(arg namespace)/${name}" />
-      <child link="${lidar_link_ns}" />
+      <parent link="${ns}${name}" />
+      <child link="${ns}${lidar_link}" />
       <origin xyz="0.0 0.0 0.03618" rpy="0 0 0" />
     </joint>
     <!-- Gazebo requires the ouster_gazebo_plugins package -->
-    <gazebo reference="$(arg namespace)/${name}">
+    <gazebo reference="${ns}${name}">
         <selfCollide>false</selfCollide>
-        <sensor name="$(arg namespace)/${name}-OS1-32" type="gpu_lidar">
+        <sensor name="${ns}${name}-OS1-32" type="gpu_lidar">
             <pose> 0 0 0 0 0 0 </pose>
             <always_on>true</always_on>
             <update_rate>${hz}</update_rate>
             <visualize>false</visualize>
-            <gz_frame_id>${lidar_link_ns}</gz_frame_id>
-            <topic>$(arg namespace)${topic_points}</topic>
+            <gz_frame_id>${ns}${lidar_link}</gz_frame_id>
+            <topic>${ns}${topic_points}</topic>
             <lidar>
                 <scan>

File: src/jackal_description/urdf/accessories/_d435.urdf.xacro (robot description, xacro)
@@ -51,14 +51,14 @@
     <joint name="${name}_joint" type="fixed">
       <xacro:insert_block name="origin" />
-      <parent link="$(arg namespace)/${parent}"/>
-      <child link="$(arg namespace)/${name}_bottom_screw_frame" />
+      <parent link="${ns}${parent}"/>
+      <child link="${ns}${name}_bottom_screw_frame" />
     </joint>
-    <link name="$(arg namespace)/${name}_bottom_screw_frame"/>
+    <link name="${ns}${name}_bottom_screw_frame"/>
     <joint name="${name}_link_joint" type="fixed">
       <origin xyz="${d435_mesh_x_offset} ${d435_cam_depth_py} ${d435_cam_depth_pz}" rpy="0 0 0"/>
-      <parent link="$(arg namespace)/${name}_bottom_screw_frame"/>
-      <child link="$(arg namespace)/${name}_link" />
+      <parent link="${ns}${name}_bottom_screw_frame"/>
+      <child link="${ns}${name}_link" />
     </joint>
-    <link name="$(arg namespace)/${name}_link">
+    <link name="${ns}${name}_link">
       <visual>
         <xacro:if value="${use_mesh}">
@@ -96,53 +96,53 @@
       <joint name="${name}_depth_joint" type="fixed">
         <origin xyz="0 0 0" rpy="0 0 0"/>
-        <parent link="$(arg namespace)/${name}_link"/>
-        <child link="$(arg namespace)/${name}_depth_frame" />
+        <parent link="${ns}${name}_link"/>
+        <child link="${ns}${name}_depth_frame" />
       </joint>
-      <link name="$(arg namespace)/${name}_depth_frame"/>
+      <link name="${ns}${name}_depth_frame"/>
       <joint name="${name}_depth_optical_joint" type="fixed">
         <origin xyz="0 0 0" rpy="${-M_PI/2} 0 ${-M_PI/2}" />
-        <parent link="$(arg namespace)/${name}_depth_frame" />
-        <child link="$(arg namespace)/${name}_depth_optical_frame" />
+        <parent link="${ns}${name}_depth_frame" />
+        <child link="${ns}${name}_depth_optical_frame" />
       </joint>
-      <link name="$(arg namespace)/${name}_depth_optical_frame"/>
+      <link name="${ns}${name}_depth_optical_frame"/>
       <!-- camera left IR joints and links -->
       <joint name="${name}_infra1_joint" type="fixed">
         <origin xyz="0 ${d435_cam_depth_to_infra1_offset} 0" rpy="0 0 0" />
-        <parent link="$(arg namespace)/${name}_link" />
-        <child link="$(arg namespace)/${name}_infra1_frame" />
+        <parent link="${ns}${name}_link" />
+        <child link="${ns}${name}_infra1_frame" />
       </joint>
-      <link name="$(arg namespace)/${name}_infra1_frame"/>
+      <link name="${ns}${name}_infra1_frame"/>
       <joint name="${name}_infra1_optical_joint" type="fixed">
         <origin xyz="0 0 0" rpy="${-M_PI/2} 0 ${-M_PI/2}" />
-        <parent link="$(arg namespace)/${name}_infra1_frame" />
-        <child link="$(arg namespace)/${name}_infra1_optical_frame" />
+        <parent link="${ns}${name}_infra1_frame" />
+        <child link="${ns}${name}_infra1_optical_frame" />
       </joint>
-      <link name="$(arg namespace)/${name}_infra1_optical_frame"/>
+      <link name="${ns}${name}_infra1_optical_frame"/>
       <!-- camera right IR joints and links -->
       <joint name="${name}_infra2_joint" type="fixed">
         <origin xyz="0 ${d435_cam_depth_to_infra2_offset} 0" rpy="0 0 0" />
-        <parent link="$(arg namespace)/${name}_link" />
-        <child link="$(arg namespace)/${name}_infra2_frame" />
+        <parent link="${ns}${name}_link" />
+        <child link="${ns}${name}_infra2_frame" />
       </joint>
-      <link name="$(arg namespace)/${name}_infra2_frame"/>
+      <link name="${ns}${name}_infra2_frame"/>
       <joint name="${name}_infra2_optical_joint" type="fixed">
         <origin xyz="0 0 0" rpy="${-M_PI/2} 0 ${-M_PI/2}" />
-        <parent link="$(arg namespace)/${name}_infra2_frame" />
-        <child link="$(arg namespace)/${name}_infra2_optical_frame" />
+        <parent link="${ns}${name}_infra2_frame" />
+        <child link="${ns}${name}_infra2_optical_frame" />
       </joint>
-      <link name="$(arg namespace)/${name}_infra2_optical_frame"/>
+      <link name="${ns}${name}_infra2_optical_frame"/>
       <!-- camera color joints and links -->
       <joint name="${name}_color_joint" type="fixed">
         <origin xyz="0 ${d435_cam_depth_to_color_offset} 0" rpy="0 0 0" />
-        <parent link="$(arg namespace)/${name}_link" />
-        <child link="$(arg namespace)/${name}_color_frame" />
+        <parent link="${ns}${name}_link" />
+        <child link="${ns}${name}_color_frame" />
       </joint>
-      <link name="$(arg namespace)/${name}_color_frame"/>
+      <link name="${ns}${name}_color_frame"/>
       <joint name="${name}_color_optical_joint" type="fixed">
         <origin xyz="0 0 0" rpy="${-M_PI/2} 0 ${-M_PI/2}" />
-        <parent link="$(arg namespace)/${name}_color_frame" />
-        <child link="$(arg namespace)/${name}_color_optical_frame" />
+        <parent link="${ns}${name}_color_frame" />
+        <child link="${ns}${name}_color_optical_frame" />
       </joint>
-      <link name="$(arg namespace)/${name}_color_optical_frame"/>
+      <link name="${ns}${name}_color_optical_frame"/>
     </xacro:if>
     <xacro:if value="${add_plug}">

File: src/jackal_description/urdf/accessories/_usb_plug.urdf.xacro (robot description, xacro)
@@ -24,8 +24,8 @@
     <joint name="${name}_joint" type="fixed">
       <xacro:insert_block name="origin" />
-      <parent link="$(arg namespace)/${parent}" />
-      <child link="$(arg namespace)/${name}_link" />
+      <parent link="${ns}${parent}" />
+      <child link="${ns}${name}_link" />
     </joint>
-    <link name="$(arg namespace)/${name}_link">
+    <link name="${ns}${name}_link">
       <visual>
         <!-- 0.044850 0.008000 0.018500 -->

File: src/jackal_description/urdf/accessories/camera_mount.urdf.xacro (robot description, xacro)
@@ -1,5 +1,5 @@
 <robot xmlns:xacro="http://www.ros.org/wiki/xacro">
   <xacro:macro name="camera_mount" params="prefix tilt:=0">
-    <link name="$(arg namespace)/${prefix}_camera_mount">
+    <link name="${ns}${prefix}_camera_mount">
       <visual>
         <origin xyz="0 0 0" rpy="1.5707 0 1.5707" />
@@ -10,5 +10,5 @@
       </visual>
     </link>
-    <link name="$(arg namespace)/${prefix}_camera_beam">
+    <link name="${ns}${prefix}_camera_beam">
       <visual>
         <origin xyz="0 0 0" rpy="0 0 1.5707" />
@@ -21,11 +21,11 @@
     <joint name="${prefix}_camera_pivot_joint" type="fixed">
       <origin xyz="0.102 0 0.008" rpy="0 ${tilt} 0" />
-      <parent link="$(arg namespace)/${prefix}_camera_mount" />
-      <child link="$(arg namespace)/${prefix}_camera_beam" />
+      <parent link="${ns}${prefix}_camera_mount" />
+      <child link="${ns}${prefix}_camera_beam" />
     </joint>
-    <gazebo reference="$(arg namespace)/${prefix}_camera_beam">
+    <gazebo reference="${ns}${prefix}_camera_beam">
       <material>Gazebo/DarkGrey</material>
     </gazebo>
-    <gazebo reference="$(arg namespace)/${prefix}_camera_mount">
+    <gazebo reference="${ns}${prefix}_camera_mount">
       <material>Gazebo/DarkGrey</material>
     </gazebo>

File: src/jackal_description/urdf/jackal.urdf.xacro (robot description, xacro)
@@ -3,4 +3,9 @@
   <xacro:property name="PI" value="3.1415926535897931" />
   <xacro:arg name="namespace" default='' />
+  <xacro:property name="ns_value" value="$(arg namespace)" />
+  <xacro:property name="ns" value="" />
+  <xacro:if value="${ns_value != ''}">
+    <xacro:property name="ns" value="${ns}/" />
+  </xacro:if>
   <!-- Jackal properties -->
   <xacro:property name="wheelbase" value="0.262" />
@@ -21,5 +26,5 @@
   <!-- Wheels macro -->
   <xacro:macro name="wheel" params="prefix mu *joint_pose">
-    <link name="$(arg namespace)/${prefix}_wheel_link">
+    <link name="${ns}${prefix}_wheel_link">
       <visual>
         <origin xyz="0 0 0" rpy="${PI/2} 0 0"/>
@@ -45,6 +50,6 @@
     </link>
     <joint name="${prefix}_wheel" type="continuous">
-      <parent link="$(arg namespace)/chassis_link"/>
-      <child link="$(arg namespace)/${prefix}_wheel_link" />
+      <parent link="${ns}chassis_link"/>
+      <child link="${ns}${prefix}_wheel_link" />
       <xacro:insert_block name="joint_pose" />
       <axis xyz="0 1 0" />
@@ -61,11 +66,11 @@
   </xacro:macro>
   <!-- Links and joints -->
-  <link name="$(arg namespace)/base_link"></link>
+  <link name="${ns}base_link"></link>
   <joint name="base_link_joint" type="fixed">
     <origin xyz="0 0 0" rpy="0 0 0" />
-    <parent link="$(arg namespace)/base_link"/>
-    <child link="$(arg namespace)/chassis_link" />
-  </joint>
-  <link name="$(arg namespace)/chassis_link">
+    <parent link="${ns}base_link"/>
+    <child link="${ns}chassis_link" />
+  </joint>
+  <link name="${ns}chassis_link">
     <visual>
       <origin xyz="0 0 ${footprint_vertical_offset}" rpy="${PI/2} 0 ${PI/2}"/>
@@ -90,5 +95,5 @@
       </inertial>
   </link>
-  <link name="$(arg namespace)/front_fender_link">
+  <link name="${ns}front_fender_link">
     <visual>
       <geometry>
@@ -98,16 +103,16 @@
     </visual>
   </link>
-  <link name="$(arg namespace)/front_fender_accessory_link"/>
+  <link name="${ns}front_fender_accessory_link"/>
   <joint name="front_fender_accessory_joint" type="fixed">
     <origin xyz="0.25629 0 0.07455" rpy="${PI} 0 0" />
-    <parent link="$(arg namespace)/front_fender_link" />
-    <child link="$(arg namespace)/front_fender_accessory_link" />
+    <parent link="${ns}front_fender_link" />
+    <child link="${ns}front_fender_accessory_link" />
   </joint>
   <joint name="front_fender_joint" type="fixed">
     <origin xyz="0 0 0" rpy="0 0 0"/>
-    <parent link="$(arg namespace)/chassis_link" />
-    <child link="$(arg namespace)/front_fender_link" />
-  </joint>
-  <link name="$(arg namespace)/rear_fender_link">
+    <parent link="${ns}chassis_link" />
+    <child link="${ns}front_fender_link" />
+  </joint>
+  <link name="${ns}rear_fender_link">
     <visual>
       <geometry>
@@ -117,14 +122,14 @@
     </visual>
   </link>
-  <link name="$(arg namespace)/rear_fender_accessory_link"/>
+  <link name="${ns}rear_fender_accessory_link"/>
   <joint name="rear_fender_accessory_joint" type="fixed">
     <origin xyz="0.25629 0 0.07455" rpy="${PI} 0 0" />
-    <parent link="$(arg namespace)/rear_fender_link" />
-    <child link="$(arg namespace)/rear_fender_accessory_link" />
+    <parent link="${ns}rear_fender_link" />
+    <child link="${ns}rear_fender_accessory_link" />
   </joint>
   <joint name="rear_fender_joint" type="fixed">
     <origin xyz="0 0 0" rpy="0 0 ${PI}"/>
-    <parent link="$(arg namespace)/chassis_link" />
-    <child link="$(arg namespace)/rear_fender_link" />
+    <parent link="${ns}chassis_link" />
+    <child link="${ns}rear_fender_link" />
   </joint>
   <!-- Wheels links and joints -->
@@ -142,5 +147,5 @@
   </xacro:wheel>
   <!-- Default Internal IMU Link -->
-  <link name="$(arg namespace)/imu_link">
+  <link name="${ns}imu_link">
     <inertial>
       <mass value="0.001"/>
@@ -150,9 +155,9 @@
   </link>
   <joint name="imu_joint" type="fixed">
-    <parent link="$(arg namespace)/chassis_link" />
-    <child link="$(arg namespace)/imu_link" />
+    <parent link="${ns}chassis_link" />
+    <child link="${ns}imu_link" />
   </joint>
   <!-- Default NAVSAT Link -->
-  <link name="$(arg namespace)/navsat_link">
+  <link name="${ns}navsat_link">
     <visual>
       <geometry>
@@ -164,24 +169,24 @@
   </link>
   <joint name="navsat_joint" type="fixed">
-    <parent link="$(arg namespace)/chassis_link" />
-    <child link="$(arg namespace)/navsat_link" />
+    <parent link="${ns}chassis_link" />
+    <child link="${ns}navsat_link" />
     <origin xyz="-0.180 0.126 0.1815" />
   </joint>
-  <link name="$(arg namespace)/mid_mount"></link>
+  <link name="${ns}mid_mount"></link>
   <joint name="mid_mount_joint" type="fixed">
-    <parent link="$(arg namespace)/chassis_link" />
-    <child link="$(arg namespace)/mid_mount" />
+    <parent link="${ns}chassis_link" />
+    <child link="${ns}mid_mount" />
     <origin xyz="0 0 ${chassis_height}" />
   </joint>
-  <link name="$(arg namespace)/rear_mount"></link>
+  <link name="${ns}rear_mount"></link>
   <joint name="rear_mount_joint" type="fixed">
-    <parent link="$(arg namespace)/mid_mount" />
-    <child link="$(arg namespace)/rear_mount" />
+    <parent link="${ns}mid_mount" />
+    <child link="${ns}rear_mount" />
     <origin xyz="${-mount_spacing} 0 0" />
   </joint>
-  <link name="$(arg namespace)/front_mount"></link>
+  <link name="${ns}front_mount"></link>
   <joint name="front_mount_joint" type="fixed">
-    <parent link="$(arg namespace)/mid_mount" />
-    <child link="$(arg namespace)/front_mount" />
+    <parent link="${ns}mid_mount" />
+    <child link="${ns}front_mount" />
     <origin xyz="${mount_spacing} 0 0" />
   </joint>
@@ -191,6 +196,6 @@
     <origin xyz="0 0 0"
             rpy="0 0 0" />
-    <parent link="$(arg namespace)/front_mount" />
-    <child link="$(arg namespace)/front_camera_mount" />
+    <parent link="${ns}front_mount" />
+    <child link="${ns}front_camera_mount" />
   </joint>
   <!-- Realsense D435 -->
